File: final_board/final_outline.sch (KiCad schematic (older format))
At the start: 0 parts

Commit message: Final changes to board
Changed lines of the file:
@@
 EESchema Schematic File Version 2
-LIBS:final_outline-rescue
 LIBS:power
 LIBS:device
@@
 LIBS:MITEVT_power
 LIBS:MITEVT_REG
+LIBS:zsr1000gta
 LIBS:final_outline-cache
 EELAYER 25 0
@@
 F0 "FRONT_PANEL" 60
 F1 "front_panel.sch" 60
-F2 "+5V" O R 3600 2850 60
+F2 "+12V" O R 3600 2850 60
 F3 "RXD" O R 3600 3050 60
 F4 "TXD" I R 3600 3150 60
@@
 F3 "+3V3" O R 6050 2150 60
 F4 "+5V" O R 6050 2550 60
+F5 "+10V" O R 6050 2800 60
 $EndSheet
 Wire Wire Line
@@
 Wire Wire Line
 	7400 3750 6450 3750
+$Comp
+L VCC #PWR04
+U 1 1 56920327
+P 6450 2750
+F 0 "#PWR04" H 6450 2600 50  0001 C CNN
+F 1 "VCC" H 6450 2900 50  0000 C CNN
+F 2 "" H 6450 2750 50  0000 C CNN
+F 3 "" H 6450 2750 50  0000 C CNN
+	1    6450 2750
+	1    0    0    -1
+$EndComp
+Wire Wire Line
+	6050 2800 6450 2800
+Wire Wire Line
+	6450 2800 6450 2750
 $EndSCHEMATC

Commit message: Fixed some routing
Changed lines of the file:
@@
 LIBS:MITEVT_power
 LIBS:MITEVT_REG
-LIBS:zsr1000gta
 LIBS:final_outline-cache
 EELAYER 25 0
@@
 F0 "FRONT_PANEL" 60
 F1 "front_panel.sch" 60
-F2 "+12V" O R 3600 2850 60
+F2 "+5V" O R 3600 2850 60
 F3 "RXD" O R 3600 3050 60
 F4 "TXD" I R 3600 3150 60
@@
 F14 "CANL" B R 6250 5100 60
 F15 "CANH" B R 6250 5000 60
-F16 "CANP" I R 6250 4900 60
-F17 "WVS_PULSE" I R 6250 4700 60
+F16 "WVS_PULSE" I R 6250 4700 60
 $EndSheet
 $Sheet
@@
 F2 "+12V" I L 4850 2150 60
 F3 "+3V3" O R 6050 2150 60
-F4 "+5V" O R 6050 2550 60
+F4 "+5V" O L 4850 2500 60
 F5 "+10V" O R 6050 2800 60
 $EndSheet
@@
 Wire Wire Line
 	4300 2150 4850 2150
-Wire Wire Line
-	4300 2000 4300 2850
-Wire Wire Line
-	4300 2850 3600 2850
 Wire Wire Line
 	3600 3050 4350 3050
@@
 	4700 1450 4700 2150
 Connection ~ 4700 2150
-Connection ~ 4300 2150
 Wire Wire Line
 	6800 1450 4700 1450
 Wire Wire Line
-	6800 1450 6800 4900
+	6800 1450 6800 3050
 Wire Wire Line
 	6800 3050 7400 3050
-Wire Wire Line
-	6800 4900 6250 4900
-Connection ~ 6800 3050
 $Comp
 L +12V #PWR02
@@
 Wire Wire Line
 	6450 2000 6450 2150
-$Comp
-L +5V #PWR03
-U 1 1 5650EA5F
-P 6450 2400
-F 0 "#PWR03" H 6450 2250 50  0001 C CNN
-F 1 "+5V" H 6450 2540 50  0000 C CNN
-F 2 "" H 6450 2400 60  0000 C CNN
-F 3 "" H 6450 2400 60  0000 C CNN
-	1    6450 2400
-	1    0    0    -1
-$EndComp
-Wire Wire Line
-	6450 2400 6450 2550
-Wire Wire Line
-	6450 2550 6050 2550
 $Sheet
 S 4750 3250 1700 950
@@
 	7400 3750 6450 3750
 $Comp
-L VCC #PWR04
+L VCC #PWR03
 U 1 1 56920327
 P 6450 2750
-F 0 "#PWR04" H 6450 2600 50  0001 C CNN
+F 0 "#PWR03" H 6450 2600 50  0001 C CNN
 F 1 "VCC" H 6450 2900 50  0000 C CNN
 F 2 "" H 6450 2750 50  0000 C CNN
@@
 Wire Wire Line
 	6450 2800 6450 2750
+Wire Wire Line
+	4300 2000 4300 2150
+Wire Wire Line
+	4850 2500 3950 2500
+Wire Wire Line
+	3950 2300 3950 2850
+Wire Wire Line
+	3950 2850 3600 2850
+Connection ~ 3950 2500
+$Comp
+L +5V #PWR04
+U 1 1 5695D325
+P 3950 2300
+F 0 "#PWR04" H 3950 2150 50  0001 C CNN
+F 1 "+5V" H 3950 2440 50  0000 C CNN
+F 2 "" H 3950 2300 50  0000 C CNN
+F 3 "" H 3950 2300 50  0000 C CNN
+	1    3950 2300
+	1    0    0    -1
+$EndComp
 $EndSCHEMATC
