File: final_board/final_outline.kicad_pcb (KiCad board)
At the start: 2 copper layers, 99.5 x 75 mm, 40 parts, among them P001 CANCONNECTOR, P002 AUXCONNECTOR, P100 ISP, P101 DEBUG_LED, U401 ISO1050, U403 LPC11C14, U501 MCP1755-33, U502 MCP1755-5, U601 LM358, U602 LM311N

Commit message: Final changes to board
Parts:
- removed C401: 10uF, Capacitors_SMD:C_0805_HandSoldering
- removed C402: 0.1uF, Capacitors_SMD:C_0603
- removed U401: ISO1050, Housings_SSOP:MSOP-8_3x3mm_Pitch0.65mm
- added C501: 10μ, Capacitors_SMD:C_0805_HandSoldering, F.Cu at (143.8, 109.2)
- added C502: .1μ, Capacitors_SMD:C_0603_HandSoldering, F.Cu at (140.0, 109.4)
- added C503: 10μ, Capacitors_SMD:C_0805_HandSoldering, F.Cu at (135.4, 99.2)
- added C504: .1μ, Capacitors_SMD:C_0603_HandSoldering, F.Cu at (135.8, 96.0)
- added C505: 10μ, Capacitors_SMD:C_0805_HandSoldering, F.Cu at (159.0, 105.8)
- added C506: .1μ, Capacitors_SMD:C_0603_HandSoldering, F.Cu at (159.0, 100.6)
- added R1: 20k, Capacitors_SMD:C_0603_HandSoldering, F.Cu at (128.4, 103.4)
- added U402: MCP2551-I/SN, Housings_SOIC:SOIC-8_3.9x4.9mm_Pitch1.27mm, F.Cu at (122.6, 100.4)
- added U503: Zsr1000gta, TO_SOT_Packages_SMD:SOT-223, F.Cu at (152.0, 102.7)
- moved C404 7.44 mm to (123.4, 92.8), turned to 0 degrees
- moved C403 5.01 mm to (122.8, 95.2), turned to 0 degrees
- moved U501 4.14 mm to (137.6, 91.6)
- moved U502 1.54 mm to (137.6, 103.6)
- moved R201 0.30 mm to (122.6, 106.6)
Connections:
- C403 pad 1: +3V3 -> +5V
- C404 pad 1: +3V3 -> +5V
- C601 pad 1: +12V -> VCC
- C602 pad 1: +12V -> VCC
- D601 pad 1: +12V -> VCC
- D603 pad 1: +12V -> VCC
- R601 pad 1: +12V -> VCC
- U601 pad 8: +12V -> VCC
- U602 pad 8: +12V -> VCC
Routing:
- net VCC: track 0.00 -> 86.1 mm, vias 0 -> 3
- net +12V: track 194.8 -> 137.0 mm, vias 7 -> 1
- net +3V3: track 70.5 -> 52.4 mm
- net +5V: track 22.8 -> 35.5 mm, vias 0 -> 2
- net GND: track 58.0 -> 45.9 mm, vias 15 -> 12
- net /Micro_Controller/CAN_TXD: track 19.0 -> 27.4 mm, vias 2 -> 0
- net /BACK_PANEL/CANL: track 26.4 -> 22.4 mm
- net /BACK_PANEL/CANH: track 26.1 -> 22.5 mm
- net Net-(R1-Pad1): track 0.00 -> 3.07 mm
- net (no net): track 0.63 -> 2.77 mm, vias 0 -> 1

Commit message: The ISP is no longer providing 12 volts
Parts:
- R201: value R -> 120
Connections:
- P100 pad 3: +12V -> +5V
Routing:
- net +12V: track 137.0 -> 51.7 mm
- net +5V: track 35.5 -> 106.1 mm
- net (no net): track 2.77 -> 5.38 mm, vias 1 -> 2
- net GND: track 45.9 -> 43.2 mm, vias 12 -> 11
Changed lines of the file:
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@@
     (thickness 1.6)
     (drawings 6)
-    (tracks 427)
+    (tracks 428)
     (zones 0)
     (modules 46)
@@
       (net 29 /FRONT_PANEL/MCU_PROG_N))
     (pad 3 thru_hole circle (at -6 0 180) (size 1.5 1.5) (drill 1.1) (layers *.Cu *.Mask F.SilkS)
-      (net 78 +12V))
+      (net 73 +5V))
     (pad "" np_thru_hole circle (at -3 4.32 180) (size 3.1 3.1) (drill 3.1) (layers *.Cu *.Mask F.SilkS))
   )
@@
       (effects (font (size 1 1) (thickness 0.15)))
     )
-    (fp_text value R (at 0 1.9) (layer F.Fab)
+    (fp_text value 120 (at 0 1.9) (layer F.Fab)
       (effects (font (size 1 1) (thickness 0.15)))
     )
@@
   (via (at 125.6 94.6) (size 0.8) (drill 0.4) (layers F.Cu B.Cu) (net 0))
   (segment (start 124.8 93.8) (end 125.6 94.6) (width 0.5) (layer B.Cu) (net 0))
+  (segment (start 160 100.6) (end 160 99.4) (width 0.5) (layer B.Cu) (net 0))
+  (via (at 161 98.4) (size 0.8) (drill 0.4) (layers F.Cu B.Cu) (net 0))
+  (segment (start 160 99.4) (end 161 98.4) (width 0.5) (layer B.Cu) (net 0))
   (segment (start 119 69) (end 119.11 69.11) (width 0.25) (layer F.Cu) (net 21))
   (segment (start 119.11 69.11) (end 119.11 70.05) (width 0.25) (layer F.Cu) (net 21))
@@
   (segment (start 141.97 70.15) (end 141.97 70.3) (width 0.25) (layer F.Cu) (net 24))
   (segment (start 139 67.18) (end 141.97 70.15) (width 0.25) (layer F.Cu) (net 24))
-  (segment (start 146.497 93.345) (end 146.497 95.303) (width 0.5) (layer F.Cu) (net 25) (status 400000))
+  (segment (start 146.497 93.345) (end 146.497 95.303) (width 0.5) (layer F.Cu) (net 25))
   (via (at 145.2 96.6) (size 0.8) (drill 0.4) (layers F.Cu B.Cu) (net 25))
   (segment (start 146.497 95.303) (end 145.2 96.6) (width 0.5) (layer F.Cu) (net 25))
-  (segment (start 160 100.6) (end 160 99.4) (width 0.5) (layer B.Cu) (net 25))
-  (via (at 161 98.4) (size 0.8) (drill 0.4) (layers F.Cu B.Cu) (net 25))
-  (segment (start 160 99.4) (end 161 98.4) (width 0.5) (layer B.Cu) (net 25))
   (segment (start 137.6 103.92) (end 137.6 100.8) (width 0.25) (layer F.Cu) (net 25))
   (segment (start 137.6 100.8) (end 139.4 99) (width 0.25) (layer F.Cu) (net 25))
@@
   (segment (start 136 68) (end 137 69) (width 0.25) (layer F.Cu) (net 72))
   (segment (start 136 65) (end 136 68) (width 0.25) (layer F.Cu) (net 72))
+  (segment (start 141.8 89.155) (end 141.8 89.45) (width 0.5) (layer F.Cu) (net 73))
+  (segment (start 141.8 89.45) (end 138.55 92.7) (width 0.5) (layer F.Cu) (net 73))
   (segment (start 137.6 95) (end 138.55 94.05) (width 0.5) (layer F.Cu) (net 73))
+  (segment (start 136.65 95) (end 137.6 95) (width 0.5) (layer F.Cu) (net 73))
   (segment (start 138.55 94.05) (end 138.55 92.7) (width 0.5) (layer F.Cu) (net 73))
   (segment (start 136.65 95) (end 136.65 92.7) (width 0.5) (layer F.Cu) (net 73))
   (segment (start 136.65 95.45) (end 136.65 95) (width 0.5) (layer F.Cu) (net 73))
-  (segment (start 136.65 95) (end 137.6 95) (width 0.5) (layer F.Cu) (net 73))
   (segment (start 136.75 95.55) (end 136.65 95.45) (width 0.5) (layer F.Cu) (net 73))
   (segment (start 136.75 96) (end 136.75 95.55) (width 0.5) (layer F.Cu) (net 73))
@@
   (segment (start 122.15 92.8) (end 122.15 95.1) (width 0.5) (layer F.Cu) (net 73))
   (segment (start 122.15 95.1) (end 122.05 95.2) (width 0.5) (layer F.Cu) (net 73))
+  (segment (start 185.88 62.25) (end 186.94066 62.25) (width 0.5) (layer F.Cu) (net 73))
+  (segment (start 186.94066 62.25) (end 187.8 63.10934) (width 0.5) (layer F.Cu) (net 73))
+  (segment (start 158.6 68.8) (end 151.6 75.8) (width 0.5) (layer F.Cu) (net 73))
+  (segment (start 187.8 63.10934) (end 187.8 65.6) (width 0.5) (layer F.Cu) (net 73))
+  (segment (start 187.8 65.6) (end 184.6 68.8) (width 0.5) (layer F.Cu) (net 73))
+  (segment (start 184.6 68.8) (end 158.6 68.8) (width 0.5) (layer F.Cu) (net 73))
+  (segment (start 144.955 86) (end 141.8 89.155) (width 0.5) (layer F.Cu) (net 73))
+  (segment (start 141.8 89.155) (end 141.8 89.155) (width 0.5) (layer F.Cu) (net 73))
+  (segment (start 141.8 89.155) (end 141.8 89.155) (width 0.5) (layer F.Cu) (net 73))
+  (segment (start 151.6 75.8) (end 151.6 84.6) (width 0.5) (layer F.Cu) (net 73))
+  (segment (start 151.6 84.6) (end 150.2 86) (width 0.5) (layer F.Cu) (net 73))
+  (segment (start 150.2 86) (end 144.955 86) (width 0.5) (layer F.Cu) (net 73))
   (segment (start 121.5 106.6) (end 121.5 106.1) (width 0.25) (layer F.Cu) (net 74))
   (segment (start 121.965 105.635) (end 121.965 103.1) (width 0.25) (layer F.Cu) (net 74))
@@
   (segment (start 146.8 111.4) (end 146.8 107.8) (width 0.5) (layer B.Cu) (net 78))
   (segment (start 136.652 112.649) (end 145.551 112.649) (width 0.5) (layer B.Cu) (net 78))
-  (segment (start 141.8 102.275) (end 143.8 104.275) (width 0.5) (layer F.Cu) (net 78))
-  (segment (start 143.8 104.275) (end 143.8 107.95) (width 0.5) (layer F.Cu) (net 78))
-  (segment (start 185.88 62.25) (end 186.94066 62.25) (width 0.5) (layer F.Cu) (net 78))
-  (segment (start 186.94066 62.25) (end 187.8 63.10934) (width 0.5) (layer F.Cu) (net 78))
-  (segment (start 158.6 68.8) (end 151.6 75.8) (width 0.5) (layer F.Cu) (net 78))
-  (segment (start 187.8 63.10934) (end 187.8 65.6) (width 0.5) (layer F.Cu) (net 78))
-  (segment (start 144.955 86) (end 141.8 89.155) (width 0.5) (layer F.Cu) (net 78))
-  (segment (start 187.8 65.6) (end 184.6 68.8) (width 0.5) (layer F.Cu) (net 78))
-  (segment (start 151.6 75.8) (end 151.6 84.6) (width 0.5) (layer F.Cu) (net 78))
-  (segment (start 151.6 84.6) (end 150.2 86) (width 0.5) (layer F.Cu) (net 78))
-  (segment (start 184.6 68.8) (end 158.6 68.8) (width 0.5) (layer F.Cu) (net 78))
-  (segment (start 150.2 86) (end 144.955 86) (width 0.5) (layer F.Cu) (net 78))
-  (segment (start 141.8 89.155) (end 141.8 102.275) (width 0.5) (layer F.Cu) (net 78))
   (segment (start 138.65 108.45) (end 136.65 106.45) (width 0.5) (layer F.Cu) (net 78))
   (segment (start 136.65 106.45) (end 136.65 104.7) (width 0.5) (layer F.Cu) (net 78))

Commit message: Removed useless trace
Routing:
- net (no net): track 5.38 -> 3.25 mm, vias 2 -> 1
Changed lines of the file:
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@@
     (links 117)
     (no_connects 0)
-    (area 102.424999 52.924999 202.075001 128.075001)
+    (area 98.806 49.875 215 135.483792)
     (thickness 1.6)
     (drawings 6)
-    (tracks 428)
+    (tracks 425)
     (zones 0)
     (modules 46)
@@
   (gr_line (start 102.5 128) (end 202 128) (layer Edge.Cuts) (width 0.15))
   (segment (start 127.381 84.455) (end 128.016 84.455) (width 0.25) (layer B.Cu) (net 0))
-  (segment (start 124.8 92.8) (end 124.8 93.8) (width 0.5) (layer B.Cu) (net 0))
-  (via (at 125.6 94.6) (size 0.8) (drill 0.4) (layers F.Cu B.Cu) (net 0))
-  (segment (start 124.8 93.8) (end 125.6 94.6) (width 0.5) (layer B.Cu) (net 0))
   (segment (start 160 100.6) (end 160 99.4) (width 0.5) (layer B.Cu) (net 0))
   (via (at 161 98.4) (size 0.8) (drill 0.4) (layers F.Cu B.Cu) (net 0))
