File: final_board/back_panel.sch (KiCad schematic (older format))
At the start: 3 parts, among them P001 CANCONNECTOR, P002 AUXCONNECTOR

Commit message: Fixed some routing
Parts:
- R201: value R -> 120
Connections:
- no-connect marks 0 -> 21
Changed lines of the file:
@@
 LIBS:MITEVT_power
 LIBS:MITEVT_REG
-LIBS:zsr1000gta
 LIBS:final_outline-cache
 EELAYER 25 0
@@
 P 2350 1100
 F 0 "R201" V 2430 1100 50  0000 C CNN
-F 1 "R" V 2350 1100 50  0000 C CNN
+F 1 "120" V 2350 1100 50  0000 C CNN
 F 2 "Resistors_SMD:R_0603_HandSoldering" V 2280 1100 30  0001 C CNN
 F 3 "" H 2350 1100 30  0000 C CNN
@@
 Text HLabel 5200 1600 0    60   Output ~ 0
 WVS-
+NoConn ~ 5200 1900
+NoConn ~ 5200 2000
+NoConn ~ 5200 1700
+NoConn ~ 5200 1500
+NoConn ~ 5200 2100
+NoConn ~ 5200 2200
+NoConn ~ 5200 2300
+NoConn ~ 5200 2400
+NoConn ~ 5200 2500
+NoConn ~ 5200 2600
+NoConn ~ 5200 2700
+NoConn ~ 5200 2800
+NoConn ~ 5200 2900
+NoConn ~ 5200 3000
+NoConn ~ 5200 3100
+NoConn ~ 5200 3200
+NoConn ~ 5200 3300
+NoConn ~ 5200 3400
+NoConn ~ 5200 3500
+NoConn ~ 5200 3600
+NoConn ~ 5200 3700
 $EndSCHEMATC

Commit message: Updated PCB by replacing old parts, fixing voltage regulator, adding test points, and general improvements
Parts:
- removed P002: AUXCONNECTOR, MITEVT_AUTOMOTIVECON:776280-1, symbol CONN_01X23
- added P002: CONN_01X14, MITEVT_AUTOMOTIVECON:776267-1, symbol CONN_01X14
- P001: footprint MITEVT_AUTOMOTIVECON:776087-1 -> MITEVT_AUTOMOTIVECON:776280-1
Connections:
- no-connect marks 21 -> 12
Changed lines of the file:
@@
 F 0 "P001" H 2350 2200 50  0000 C CNN
 F 1 "CANCONNECTOR" H 2350 1700 50  0000 C CNN
-F 2 "MITEVT_AUTOMOTIVECON:776087-1" H 2350 750 60  0001 C CNN
+F 2 "MITEVT_AUTOMOTIVECON:776280-1" H 2350 750 60  0001 C CNN
 F 3 "" H 2350 750 60  0000 C CNN
 	1    2350 1950
-	1    0    0    -1
-$EndComp
-$Comp
-L CONN_01X23 P002
-U 1 1 56352B23
-P 5400 2600
-F 0 "P002" H 5400 3800 50  0000 C CNN
-F 1 "AUXCONNECTOR" V 5500 2600 50  0000 C CNN
-F 2 "MITEVT_AUTOMOTIVECON:776280-1" H 5400 2600 60  0001 C CNN
-F 3 "" H 5400 2600 60  0000 C CNN
-	1    5400 2600
 	1    0    0    -1
 $EndComp
@@
 Connection ~ 3100 1800
 Connection ~ 1600 1800
-Text HLabel 5200 1800 0    60   Output ~ 0
+Text HLabel 4500 2400 0    60   Output ~ 0
 WVS+
-Text HLabel 5200 1600 0    60   Output ~ 0
+Text HLabel 4500 2200 0    60   Output ~ 0
 WVS-
-NoConn ~ 5200 1900
-NoConn ~ 5200 2000
-NoConn ~ 5200 1700
-NoConn ~ 5200 1500
-NoConn ~ 5200 2100
-NoConn ~ 5200 2200
-NoConn ~ 5200 2300
-NoConn ~ 5200 2400
-NoConn ~ 5200 2500
-NoConn ~ 5200 2600
-NoConn ~ 5200 2700
-NoConn ~ 5200 2800
-NoConn ~ 5200 2900
-NoConn ~ 5200 3000
-NoConn ~ 5200 3100
-NoConn ~ 5200 3200
-NoConn ~ 5200 3300
-NoConn ~ 5200 3400
-NoConn ~ 5200 3500
-NoConn ~ 5200 3600
-NoConn ~ 5200 3700
+$Comp
+L CONN_01X14 P002
+U 1 1 58276BDD
+P 4700 2750
+F 0 "P002" H 4700 3500 50  0000 C CNN
+F 1 "CONN_01X14" V 4800 2750 50  0000 C CNN
+F 2 "MITEVT_AUTOMOTIVECON:776267-1" H 4700 2750 50  0001 C CNN
+F 3 "" H 4700 2750 50  0000 C CNN
+	1    4700 2750
+	1    0    0    -1
+$EndComp
+NoConn ~ 4500 2100
+NoConn ~ 4500 2300
+NoConn ~ 4500 2500
+NoConn ~ 4500 2600
+NoConn ~ 4500 2700
+NoConn ~ 4500 2800
+NoConn ~ 4500 2900
+NoConn ~ 4500 3000
+NoConn ~ 4500 3100
+NoConn ~ 4500 3200
+NoConn ~ 4500 3300
+NoConn ~ 4500 3400
 $EndSCHEMATC
