File: final_board/mcu.sch (KiCad schematic (older format))
At the start: 10 parts, among them U401 ISO1050, U403 LPC11C14

Commit message: Changed CAN Chip, added capacitors, added reference
Parts:
- removed C401: 10uF, Capacitors_SMD:C_0805_HandSoldering, symbol C_Small
- removed C402: 0.1uF, Capacitors_SMD:C_0603_HandSoldering, symbol C_Small
- removed U401: ISO1050, Housings_SSOP:MSOP-8_3x3mm_Pitch0.65mm, symbol ISO1050
- added R1: 20k, Capacitors_SMD:C_0603_HandSoldering, symbol R
- added U402: MCP2551-I/SN, Housings_SOIC:SOIC-8_3.9x4.9mm_Pitch1.27mm, symbol MCP2551-I/SN
Connections:
- net labels removed: +5V
- wire segments 69 -> 63
- no-connect marks 2 -> 3
Other:
- moved on the sheet: C403, C404
Changed lines of the file:
@@
 EESchema Schematic File Version 2
-LIBS:final_outline-rescue
 LIBS:power
 LIBS:device
@@
 	1    0    0    -1
 $EndComp
-$Comp
-L ISO1050 U401
-U 1 1 563E22B3
-P 3250 4950
-F 0 "U401" H 2900 5300 60  0000 C CNN
-F 1 "ISO1050" H 3550 5300 60  0000 C CNN
-F 2 "Housings_SSOP:MSOP-8_3x3mm_Pitch0.65mm" H 3550 5300 60  0001 C CNN
-F 3 "" H 3550 5300 60  0000 C CNN
-	1    3250 4950
-	-1   0    0    -1
-$EndComp
+Text HLabel 2350 5050 0    60   BiDi ~ 0
+CANL
 Text HLabel 2350 4850 0    60   BiDi ~ 0
-CANL
-Text HLabel 2350 5050 0    60   BiDi ~ 0
 CANH
 $Comp
 L GND #PWR08
 U 1 1 563E2693
-P 3350 5800
-F 0 "#PWR08" H 3350 5550 50  0001 C CNN
-F 1 "GND" H 3350 5650 50  0000 C CNN
-F 2 "" H 3350 5800 60  0000 C CNN
-F 3 "" H 3350 5800 60  0000 C CNN
-	1    3350 5800
+P 4100 5700
+F 0 "#PWR08" H 4100 5450 50  0001 C CNN
+F 1 "GND" H 4100 5550 50  0000 C CNN
+F 2 "" H 4100 5700 60  0000 C CNN
+F 3 "" H 4100 5700 60  0000 C CNN
+	1    4100 5700
 	1    0    0    -1
 $EndComp
@@
 L GND #PWR09
 U 1 1 563E26E3
-P 3150 5800
-F 0 "#PWR09" H 3150 5550 50  0001 C CNN
-F 1 "GND" H 3150 5650 50  0000 C CNN
-F 2 "" H 3150 5800 60  0000 C CNN
-F 3 "" H 3150 5800 60  0000 C CNN
-	1    3150 5800
-	1    0    0    -1
-$EndComp
-$Comp
-L C_Small C401
-U 1 1 563E2793
-P 2400 4300
-F 0 "C401" H 2410 4370 50  0000 L CNN
-F 1 "10uF" H 2410 4220 50  0000 L CNN
-F 2 "Capacitors_SMD:C_0805_HandSoldering" H 2400 4300 60  0001 C CNN
-F 3 "" H 2400 4300 60  0000 C CNN
-	1    2400 4300
-	1    0    0    -1
-$EndComp
-$Comp
-L C_Small C402
-U 1 1 563E282A
-P 2850 4300
-F 0 "C402" H 2860 4370 50  0000 L CNN
-F 1 "0.1uF" H 2860 4220 50  0000 L CNN
-F 2 "Capacitors_SMD:C_0603_HandSoldering" H 2850 4300 60  0001 C CNN
-F 3 "" H 2850 4300 60  0000 C CNN
-	1    2850 4300
+P 3250 5750
+F 0 "#PWR09" H 3250 5500 50  0001 C CNN
+F 1 "GND" H 3250 5600 50  0000 C CNN
+F 2 "" H 3250 5750 60  0000 C CNN
+F 3 "" H 3250 5750 60  0000 C CNN
+	1    3250 5750
 	1    0    0    -1
 $EndComp
@@
 L C_Small C403
 U 1 1 563E286E
-P 3650 4300
-F 0 "C403" H 3660 4370 50  0000 L CNN
-F 1 "0.1uF" H 3660 4220 50  0000 L CNN
-F 2 "Capacitors_SMD:C_0603_HandSoldering" H 3650 4300 60  0001 C CNN
-F 3 "" H 3650 4300 60  0000 C CNN
-	1    3650 4300
+P 3550 4300
+F 0 "C403" H 3560 4370 50  0000 L CNN
+F 1 "0.1uF" H 3560 4220 50  0000 L CNN
+F 2 "Capacitors_SMD:C_0603_HandSoldering" H 3550 4300 60  0001 C CNN
+F 3 "" H 3550 4300 60  0000 C CNN
+	1    3550 4300
 	1    0    0    -1
 $EndComp
@@
 L C_Small C404
 U 1 1 563E28A1
-P 4100 4300
-F 0 "C404" H 4110 4370 50  0000 L CNN
-F 1 "10uF" H 4110 4220 50  0000 L CNN
-F 2 "Capacitors_SMD:C_0805_HandSoldering" H 4100 4300 60  0001 C CNN
-F 3 "" H 4100 4300 60  0000 C CNN
-	1    4100 4300
+P 4000 4300
+F 0 "C404" H 4010 4370 50  0000 L CNN
+F 1 "10uF" H 4010 4220 50  0000 L CNN
+F 2 "Capacitors_SMD:C_0805_HandSoldering" H 4000 4300 60  0001 C CNN
+F 3 "" H 4000 4300 60  0000 C CNN
+	1    4000 4300
 	1    0    0    -1
 $EndComp
 $Comp
 L GND #PWR010
-U 1 1 563E2981
-P 2400 4650
-F 0 "#PWR010" H 2400 4400 50  0001 C CNN
-F 1 "GND" H 2400 4500 50  0000 C CNN
-F 2 "" H 2400 4650 60  0000 C CNN
-F 3 "" H 2400 4650 60  0000 C CNN
-	1    2400 4650
-	1    0    0    -1
-$EndComp
-$Comp
-L GND #PWR011
 U 1 1 563E2AAC
-P 4100 4550
-F 0 "#PWR011" H 4100 4300 50  0001 C CNN
-F 1 "GND" H 4100 4400 50  0000 C CNN
-F 2 "" H 4100 4550 60  0000 C CNN
-F 3 "" H 4100 4550 60  0000 C CNN
-	1    4100 4550
+P 4000 4550
+F 0 "#PWR010" H 4000 4300 50  0001 C CNN
+F 1 "GND" H 4000 4400 50  0000 C CNN
+F 2 "" H 4000 4550 60  0000 C CNN
+F 3 "" H 4000 4550 60  0000 C CNN
+	1    4000 4550
 	1    0    0    -1
 $EndComp
@@
 PIO2_4
 $Comp
-L GND #PWR012
+L GND #PWR011
 U 1 1 563E497F
 P 6250 6200
-F 0 "#PWR012" H 6250 5950 50  0001 C CNN
+F 0 "#PWR011" H 6250 5950 50  0001 C CNN
 F 1 "GND" H 6250 6050 50  0000 C CNN
 F 2 "" H 6250 6200 60  0000 C CNN
@@
 $EndComp
 $Comp
-L GND #PWR013
+L GND #PWR012
 U 1 1 563E4F46
 P 6950 1650
-F 0 "#PWR013" H 6950 1400 50  0001 C CNN
+F 0 "#PWR012" H 6950 1400 50  0001 C CNN
 F 1 "GND" H 6950 1500 50  0000 C CNN
 F 2 "" H 6950 1650 60  0000 C CNN
@@
 LED0
 $Comp
-L +3.3V #PWR014
+L +3.3V #PWR013
 U 1 1 5647852E
 P 3450 1750
-F 0 "#PWR014" H 3450 1600 50  0001 C CNN
+F 0 "#PWR013" H 3450 1600 50  0001 C CNN
 F 1 "+3.3V" H 3450 1890 50  0000 C CNN
 F 2 "" H 3450 1750 60  0000 C CNN
@@
 $EndComp
 $Comp
-L +3.3V #PWR015
+L +3.3V #PWR014
 U 1 1 56478628
 P 4650 1750
-F 0 "#PWR015" H 4650 1600 50  0001 C CNN
+F 0 "#PWR014" H 4650 1600 50  0001 C CNN
 F 1 "+3.3V" H 4650 1890 50  0000 C CNN
 F 2 "" H 4650 1750 60  0000 C CNN
@@
 $EndComp
 $Comp
-L +3.3V #PWR016
+L +3.3V #PWR015
 U 1 1 56478697
 P 6250 1000
-F 0 "#PWR016" H 6250 850 50  0001 C CNN
+F 0 "#PWR015" H 6250 850 50  0001 C CNN
 F 1 "+3.3V" H 6250 1140 50  0000 C CNN
 F 2 "" H 6250 1000 60  0000 C CNN
@@
 $EndComp
 $Comp
-L +3.3V #PWR017
+L +3.3V #PWR016
 U 1 1 56478953
-P 3350 3700
-F 0 "#PWR017" H 3350 3550 50  0001 C CNN
-F 1 "+3.3V" H 3350 3840 50  0000 C CNN
-F 2 "" H 3350 3700 60  0000 C CNN
-F 3 "" H 3350 3700 60  0000 C CNN
-	1    3350 3700
-	1    0    0    -1
-$EndComp
-$Comp
-L +5V #PWR018
-U 1 1 564789D8
-P 2650 3650
-F 0 "#PWR018" H 2650 3500 50  0001 C CNN
-F 1 "+5V" H 2650 3790 50  0000 C CNN
-F 2 "" H 2650 3650 60  0000 C CNN
-F 3 "" H 2650 3650 60  0000 C CNN
-	1    2650 3650
+P 3250 3700
+F 0 "#PWR016" H 3250 3550 50  0001 C CNN
+F 1 "+3.3V" H 3250 3840 50  0000 C CNN
+F 2 "" H 3250 3700 60  0000 C CNN
+F 3 "" H 3250 3700 60  0000 C CNN
+	1    3250 3700
 	1    0    0    -1
 $EndComp
@@
 PIO1_3
 Wire Wire Line
-	4950 4750 3850 4750
-Wire Wire Line
-	3850 4850 4950 4850
-Wire Wire Line
-	2650 4850 2350 4850
-Wire Wire Line
-	2650 5050 2350 5050
-Wire Wire Line
-	3350 5450 3350 5800
-Wire Wire Line
-	3150 5450 3150 5800
-Wire Wire Line
-	3150 3650 3150 4450
-Wire Wire Line
-	3150 3650 2650 3650
-Wire Wire Line
-	2400 4200 2400 3900
-Wire Wire Line
-	2400 3900 3150 3900
-Wire Wire Line
-	2850 3900 2850 4200
-Wire Wire Line
-	2400 4400 2400 4650
-Wire Wire Line
-	2400 4500 2850 4500
-Wire Wire Line
-	2850 4500 2850 4400
-Connection ~ 2400 4500
-Connection ~ 3150 3900
-Connection ~ 2850 3900
-Wire Wire Line
-	3350 3700 3350 4450
-Wire Wire Line
-	3350 3900 4100 3900
-Wire Wire Line
-	3650 3900 3650 4200
-Wire Wire Line
-	4100 3900 4100 4200
-Connection ~ 3650 3900
-Wire Wire Line
-	3650 4400 3650 4500
-Wire Wire Line
-	3650 4500 4100 4500
-Wire Wire Line
-	4100 4500 4100 4400
-Wire Wire Line
-	4100 4450 4100 4550
-Connection ~ 4100 4450
-Connection ~ 3350 3900
+	3750 4750 4950 4750
+Wire Wire Line
+	3750 4850 4950 4850
+Wire Wire Line
+	2350 4850 2750 4850
+Wire Wire Line
+	2350 5050 2750 5050
+Wire Wire Line
+	3250 3700 3250 4550
+Wire Wire Line
+	3550 3900 3550 4200
+Wire Wire Line
+	4000 3900 4000 4200
+Connection ~ 3550 3900
+Wire Wire Line
+	3550 4400 3550 4500
+Wire Wire Line
+	3550 4500 4000 4500
+Wire Wire Line
+	4000 4500 4000 4400
+Wire Wire Line
+	4000 4450 4000 4550
+Connection ~ 4000 4450
+Connection ~ 3250 3900
 Wire Wire Line
 	4950 4050 4650 4050
@@
 Text Label 4350 3450 0    60   ~ 0
 PIO1_0
+$Comp
+L MCP2551-I/SN U402
+U 1 1 569183E1
+P 3250 4950
+F 0 "U402" H 2850 5300 50  0000 L CNN
+F 1 "MCP2551-I/SN" H 3350 5300 50  0000 L CNN
+F 2 "Housings_SOIC:SOIC-8_3.9x4.9mm_Pitch1.27mm" H 3250 4950 50  0001 C CIN
+F 3 "" H 3250 4950 50  0000 C CNN
+	1    3250 4950
+	-1   0    0    -1
+$EndComp
+Wire Wire Line
+	3250 5350 3250 5750
+Wire Wire Line
+	3250 3900 4000 3900
+NoConn ~ 3750 5150
+$Comp
+L R R1
+U 1 1 56918BC9
+P 4100 5400
+F 0 "R1" V 4180 5400 50  0000 C CNN
+F 1 "20k" V 4100 5400 50  0000 C CNN
+F 2 "Capacitors_SMD:C_0603_HandSoldering" V 4030 5400 50  0001 C CNN
+F 3 "" H 4100 5400 50  0000 C CNN
+	1    4100 5400
+	1    0    0    -1
+$EndComp
+Wire Wire Line
+	3750 5050 4100 5050
+Wire Wire Line
+	4100 5050 4100 5250
+Wire Wire Line
+	4100 5550 4100 5700
 $EndSCHEMATC

Commit message: Final changes to board
Connections:
- net +3V3: no longer C403.1, C404.1, U402.3 (VDD)
- net at U402.5 (Vref): no longer R1.1
- net at U402.8 (Rs): now also R1.1
- new net +5V: C403.1, C404.1, U402.3 (VDD)
Changed lines of the file:
@@
 LIBS:MITEVT_power
 LIBS:MITEVT_REG
+LIBS:zsr1000gta
 LIBS:final_outline-cache
 EELAYER 25 0
@@
 CANH
 $Comp
-L GND #PWR08
+L GND #PWR09
 U 1 1 563E2693
 P 4100 5700
-F 0 "#PWR08" H 4100 5450 50  0001 C CNN
+F 0 "#PWR09" H 4100 5450 50  0001 C CNN
 F 1 "GND" H 4100 5550 50  0000 C CNN
 F 2 "" H 4100 5700 60  0000 C CNN
@@
 $EndComp
 $Comp
-L GND #PWR09
+L GND #PWR010
 U 1 1 563E26E3
 P 3250 5750
-F 0 "#PWR09" H 3250 5500 50  0001 C CNN
+F 0 "#PWR010" H 3250 5500 50  0001 C CNN
 F 1 "GND" H 3250 5600 50  0000 C CNN
 F 2 "" H 3250 5750 60  0000 C CNN
@@
 $EndComp
 $Comp
-L GND #PWR010
+L GND #PWR011
 U 1 1 563E2AAC
 P 4000 4550
-F 0 "#PWR010" H 4000 4300 50  0001 C CNN
+F 0 "#PWR011" H 4000 4300 50  0001 C CNN
 F 1 "GND" H 4000 4400 50  0000 C CNN
 F 2 "" H 4000 4550 60  0000 C CNN
@@
 PIO2_4
 $Comp
-L GND #PWR011
+L GND #PWR012
 U 1 1 563E497F
 P 6250 6200
-F 0 "#PWR011" H 6250 5950 50  0001 C CNN
+F 0 "#PWR012" H 6250 5950 50  0001 C CNN
 F 1 "GND" H 6250 6050 50  0000 C CNN
 F 2 "" H 6250 6200 60  0000 C CNN
@@
 $EndComp
 $Comp
-L GND #PWR012
+L GND #PWR013
 U 1 1 563E4F46
 P 6950 1650
-F 0 "#PWR012" H 6950 1400 50  0001 C CNN
+F 0 "#PWR013" H 6950 1400 50  0001 C CNN
 F 1 "GND" H 6950 1500 50  0000 C CNN
 F 2 "" H 6950 1650 60  0000 C CNN
@@
 LED0
 $Comp
-L +3.3V #PWR013
+L +3.3V #PWR014
 U 1 1 5647852E
 P 3450 1750
-F 0 "#PWR013" H 3450 1600 50  0001 C CNN
+F 0 "#PWR014" H 3450 1600 50  0001 C CNN
 F 1 "+3.3V" H 3450 1890 50  0000 C CNN
 F 2 "" H 3450 1750 60  0000 C CNN
@@
 $EndComp
 $Comp
-L +3.3V #PWR014
+L +3.3V #PWR015
 U 1 1 56478628
 P 4650 1750
-F 0 "#PWR014" H 4650 1600 50  0001 C CNN
+F 0 "#PWR015" H 4650 1600 50  0001 C CNN
 F 1 "+3.3V" H 4650 1890 50  0000 C CNN
 F 2 "" H 4650 1750 60  0000 C CNN
@@
 $EndComp
 $Comp
-L +3.3V #PWR015
+L +3.3V #PWR016
 U 1 1 56478697
 P 6250 1000
-F 0 "#PWR015" H 6250 850 50  0001 C CNN
+F 0 "#PWR016" H 6250 850 50  0001 C CNN
 F 1 "+3.3V" H 6250 1140 50  0000 C CNN
 F 2 "" H 6250 1000 60  0000 C CNN
 F 3 "" H 6250 1000 60  0000 C CNN
 	1    6250 1000
-	1    0    0    -1
-$EndComp
-$Comp
-L +3.3V #PWR016
-U 1 1 56478953
-P 3250 3700
-F 0 "#PWR016" H 3250 3550 50  0001 C CNN
-F 1 "+3.3V" H 3250 3840 50  0000 C CNN
-F 2 "" H 3250 3700 60  0000 C CNN
-F 3 "" H 3250 3700 60  0000 C CNN
-	1    3250 3700
 	1    0    0    -1
 $EndComp
@@
 Wire Wire Line
 	3250 3900 4000 3900
-NoConn ~ 3750 5150
 $Comp
 L R R1
@@
 $EndComp
 Wire Wire Line
-	3750 5050 4100 5050
-Wire Wire Line
-	4100 5050 4100 5250
-Wire Wire Line
 	4100 5550 4100 5700
+NoConn ~ 3750 5050
+Wire Wire Line
+	3750 5150 4100 5150
+Wire Wire Line
+	4100 5150 4100 5250
+$Comp
+L +5V #PWR017
+U 1 1 56917D77
+P 3250 3700
+F 0 "#PWR017" H 3250 3550 50  0001 C CNN
+F 1 "+5V" H 3250 3840 50  0000 C CNN
+F 2 "" H 3250 3700 50  0000 C CNN
+F 3 "" H 3250 3700 50  0000 C CNN
+	1    3250 3700
+	1    0    0    -1
+$EndComp
 $EndSCHEMATC

Commit message: Fixed some routing
Connections:
- no-connect marks 3 -> 30
Changed lines of the file:
@@
 LIBS:MITEVT_power
 LIBS:MITEVT_REG
-LIBS:zsr1000gta
 LIBS:final_outline-cache
 EELAYER 25 0
@@
 	1    0    0    -1
 $EndComp
+NoConn ~ 7600 2600
+NoConn ~ 7600 2700
+NoConn ~ 7600 2800
+NoConn ~ 7600 2900
+NoConn ~ 7600 3100
+NoConn ~ 7600 3300
+NoConn ~ 7600 3400
+NoConn ~ 7600 3500
+NoConn ~ 7600 3600
+NoConn ~ 7600 3800
+NoConn ~ 7600 3900
+NoConn ~ 7600 4150
+NoConn ~ 7600 4350
+NoConn ~ 7600 4850
+NoConn ~ 7600 5150
+NoConn ~ 4950 5250
+NoConn ~ 4950 5150
+NoConn ~ 4950 5050
+NoConn ~ 4950 4950
+NoConn ~ 4950 4650
+NoConn ~ 4950 4550
+NoConn ~ 4950 4050
+NoConn ~ 4950 3950
+NoConn ~ 4950 3850
+NoConn ~ 4950 3650
+NoConn ~ 4950 3550
+NoConn ~ 4950 3350
 $EndSCHEMATC
