File: final_board/wvs_conditioner.sch (KiCad schematic (older format))
At the start: 15 parts, among them U601 LM358, U602 LM311N

Commit message: Final changes to board
Connections:
- net +12V renamed VCC
Changed lines of the file:
@@
 EESchema Schematic File Version 2
-LIBS:final_outline-rescue
 LIBS:power
 LIBS:device
@@
 LIBS:MITEVT_power
 LIBS:MITEVT_REG
+LIBS:zsr1000gta
 LIBS:final_outline-cache
 EELAYER 25 0
@@
 $EndComp
 $Comp
-L GND #PWR022
+L GND #PWR026
 U 1 1 5650E391
 P 3500 6150
-F 0 "#PWR022" H 3500 5900 50  0001 C CNN
+F 0 "#PWR026" H 3500 5900 50  0001 C CNN
 F 1 "GND" H 3500 6000 50  0000 C CNN
 F 2 "" H 3500 6150 60  0000 C CNN
@@
 $EndComp
 $Comp
-L GND #PWR023
+L GND #PWR027
 U 1 1 5650E3B4
 P 3900 5150
-F 0 "#PWR023" H 3900 4900 50  0001 C CNN
+F 0 "#PWR027" H 3900 4900 50  0001 C CNN
 F 1 "GND" H 3900 5000 50  0000 C CNN
 F 2 "" H 3900 5150 60  0000 C CNN
@@
 	1    0    0    -1
 $EndComp
-$Comp
-L +12V #PWR024
-U 1 1 5650E3E1
-P 3500 4650
-F 0 "#PWR024" H 3500 4500 50  0001 C CNN
-F 1 "+12V" H 3500 4790 50  0000 C CNN
-F 2 "" H 3500 4650 60  0000 C CNN
-F 3 "" H 3500 4650 60  0000 C CNN
-	1    3500 4650
-	1    0    0    -1
-$EndComp
-$Comp
-L +12V #PWR025
-U 1 1 5650E402
-P 2700 4800
-F 0 "#PWR025" H 2700 4650 50  0001 C CNN
-F 1 "+12V" H 2700 4940 50  0000 C CNN
-F 2 "" H 2700 4800 60  0000 C CNN
-F 3 "" H 2700 4800 60  0000 C CNN
-	1    2700 4800
-	1    0    0    -1
-$EndComp
 Wire Wire Line
 	3500 5800 3500 6150
@@
 	2700 4800 2700 4950
 $Comp
-L GND #PWR026
+L GND #PWR028
 U 1 1 5650E4A0
 P 2700 6000
-F 0 "#PWR026" H 2700 5750 50  0001 C CNN
+F 0 "#PWR028" H 2700 5750 50  0001 C CNN
 F 1 "GND" H 2700 5850 50  0000 C CNN
 F 2 "" H 2700 6000 60  0000 C CNN
@@
 vref
 $Comp
-L GND #PWR027
+L GND #PWR029
 U 1 1 5650E751
 P 6800 3500
-F 0 "#PWR027" H 6800 3250 50  0001 C CNN
+F 0 "#PWR029" H 6800 3250 50  0001 C CNN
 F 1 "GND" H 6800 3350 50  0000 C CNN
 F 2 "" H 6800 3500 60  0000 C CNN
@@
 Connection ~ 7700 2850
 $Comp
-L +3.3V #PWR028
+L +3.3V #PWR030
 U 1 1 5650E818
 P 7700 2200
-F 0 "#PWR028" H 7700 2050 50  0001 C CNN
+F 0 "#PWR030" H 7700 2050 50  0001 C CNN
 F 1 "+3.3V" H 7700 2340 50  0000 C CNN
 F 2 "" H 7700 2200 60  0000 C CNN
@@
 $EndComp
 $Comp
-L GND #PWR029
+L GND #PWR031
 U 1 1 5650E8BE
 P 7150 1700
-F 0 "#PWR029" H 7150 1450 50  0001 C CNN
+F 0 "#PWR031" H 7150 1450 50  0001 C CNN
 F 1 "GND" H 7150 1550 50  0000 C CNN
 F 2 "" H 7150 1700 60  0000 C CNN
@@
 Wire Wire Line
 	6800 1150 6800 2550
-$Comp
-L +12V #PWR030
-U 1 1 5650E924
-P 6800 1150
-F 0 "#PWR030" H 6800 1000 50  0001 C CNN
-F 1 "+12V" H 6800 1290 50  0000 C CNN
-F 2 "" H 6800 1150 60  0000 C CNN
-F 3 "" H 6800 1150 60  0000 C CNN
-	1    6800 1150
-	1    0    0    -1
-$EndComp
 Connection ~ 6800 1300
 Text HLabel 5550 2750 0    60   Input ~ 0
@@
 	6350 2300 6350 2750
 Connection ~ 6350 2750
-$Comp
-L +12V #PWR031
-U 1 1 5650F105
-P 6450 3250
-F 0 "#PWR031" H 6450 3100 50  0001 C CNN
-F 1 "+12V" H 6450 3390 50  0000 C CNN
-F 2 "" H 6450 3250 60  0000 C CNN
-F 3 "" H 6450 3250 60  0000 C CNN
-	1    6450 3250
-	1    0    0    -1
-$EndComp
 Wire Wire Line
 	6400 1450 6400 1800
@@
 Wire Wire Line
 	6400 1000 6400 1150
-$Comp
-L +12V #PWR033
-U 1 1 5650F6E0
-P 6400 1000
-F 0 "#PWR033" H 6400 850 50  0001 C CNN
-F 1 "+12V" H 6400 1140 50  0000 C CNN
-F 2 "" H 6400 1000 60  0000 C CNN
-F 3 "" H 6400 1000 60  0000 C CNN
-	1    6400 1000
-	1    0    0    -1
-$EndComp
 Wire Wire Line
 	6450 3250 6450 3350
@@
 Connection ~ 6450 3850
 $Comp
-L GND #PWR034
+L GND #PWR033
 U 1 1 5650F87C
 P 6450 4400
-F 0 "#PWR034" H 6450 4150 50  0001 C CNN
+F 0 "#PWR033" H 6450 4150 50  0001 C CNN
 F 1 "GND" H 6450 4250 50  0000 C CNN
 F 2 "" H 6450 4400 60  0000 C CNN
@@
 Connection ~ 2950 5400
 $Comp
-L GND #PWR035
+L GND #PWR034
 U 1 1 56634664
 P 2950 5850
-F 0 "#PWR035" H 2950 5600 50  0001 C CNN
+F 0 "#PWR034" H 2950 5600 50  0001 C CNN
 F 1 "GND" H 2950 5700 50  0000 C CNN
 F 2 "" H 2950 5850 50  0000 C CNN
@@
 Wire Wire Line
 	7200 3150 7200 2950
+$Comp
+L VCC #PWR035
+U 1 1 56920678
+P 6400 1000
+F 0 "#PWR035" H 6400 850 50  0001 C CNN
+F 1 "VCC" H 6400 1150 50  0000 C CNN
+F 2 "" H 6400 1000 50  0000 C CNN
+F 3 "" H 6400 1000 50  0000 C CNN
+	1    6400 1000
+	1    0    0    -1
+$EndComp
+$Comp
+L VCC #PWR036
+U 1 1 569206B9
+P 6800 1150
+F 0 "#PWR036" H 6800 1000 50  0001 C CNN
+F 1 "VCC" H 6800 1300 50  0000 C CNN
+F 2 "" H 6800 1150 50  0000 C CNN
+F 3 "" H 6800 1150 50  0000 C CNN
+	1    6800 1150
+	1    0    0    -1
+$EndComp
+$Comp
+L VCC #PWR037
+U 1 1 569207FD
+P 6450 3250
+F 0 "#PWR037" H 6450 3100 50  0001 C CNN
+F 1 "VCC" H 6450 3400 50  0000 C CNN
+F 2 "" H 6450 3250 50  0000 C CNN
+F 3 "" H 6450 3250 50  0000 C CNN
+	1    6450 3250
+	1    0    0    -1
+$EndComp
+$Comp
+L VCC #PWR038
+U 1 1 56920898
+P 2700 4800
+F 0 "#PWR038" H 2700 4650 50  0001 C CNN
+F 1 "VCC" H 2700 4950 50  0000 C CNN
+F 2 "" H 2700 4800 50  0000 C CNN
+F 3 "" H 2700 4800 50  0000 C CNN
+	1    2700 4800
+	1    0    0    -1
+$EndComp
+$Comp
+L VCC #PWR039
+U 1 1 569208D9
+P 3500 4650
+F 0 "#PWR039" H 3500 4500 50  0001 C CNN
+F 1 "VCC" H 3500 4800 50  0000 C CNN
+F 2 "" H 3500 4650 50  0000 C CNN
+F 3 "" H 3500 4650 50  0000 C CNN
+	1    3500 4650
+	1    0    0    -1
+$EndComp
 $EndSCHEMATC

Commit message: Resistor values changed from 1k to 100k
Parts:
- R601, R602: value 1k -> 100k
Changed lines of the file:
@@
 P 2700 5100
 F 0 "R601" V 2780 5100 50  0000 C CNN
-F 1 "1k" V 2700 5100 50  0000 C CNN
+F 1 "100k" V 2700 5100 50  0000 C CNN
 F 2 "Resistors_SMD:R_0603_HandSoldering" V 2630 5100 30  0001 C CNN
 F 3 "" H 2700 5100 30  0000 C CNN
@@
 P 2700 5700
 F 0 "R602" V 2780 5700 50  0000 C CNN
-F 1 "1k" V 2700 5700 50  0000 C CNN
+F 1 "100k" V 2700 5700 50  0000 C CNN
 F 2 "Resistors_SMD:R_0603_HandSoldering" V 2630 5700 30  0001 C CNN
 F 3 "" H 2700 5700 30  0000 C CNN

Commit message: Updated PCB by replacing old parts, fixing voltage regulator, adding test points, and general improvements
Parts:
- added W01, W02, W03: TEST_1P, MITEVT_TP:smd_test_pad, symbol TEST_1P
Connections:
- net WVS+: now also W01.1
- net WVS-: now also W02.1
- net WVS_PULSE: now also W03.1
Changed lines of the file:
@@
 $EndComp
 $Comp
-L GND #PWR028
+L GND #PWR038
 U 1 1 5650E391
 P 3500 6150
-F 0 "#PWR028" H 3500 5900 50  0001 C CNN
+F 0 "#PWR038" H 3500 5900 50  0001 C CNN
 F 1 "GND" H 3500 6000 50  0000 C CNN
 F 2 "" H 3500 6150 60  0000 C CNN
@@
 $EndComp
 $Comp
-L GND #PWR029
+L GND #PWR039
 U 1 1 5650E3B4
 P 3900 5150
-F 0 "#PWR029" H 3900 4900 50  0001 C CNN
+F 0 "#PWR039" H 3900 4900 50  0001 C CNN
 F 1 "GND" H 3900 5000 50  0000 C CNN
 F 2 "" H 3900 5150 60  0000 C CNN
@@
 	2700 4800 2700 4950
 $Comp
-L GND #PWR030
+L GND #PWR040
 U 1 1 5650E4A0
 P 2700 6000
-F 0 "#PWR030" H 2700 5750 50  0001 C CNN
+F 0 "#PWR040" H 2700 5750 50  0001 C CNN
 F 1 "GND" H 2700 5850 50  0000 C CNN
 F 2 "" H 2700 6000 60  0000 C CNN
@@
 vref
 $Comp
-L GND #PWR031
+L GND #PWR041
 U 1 1 5650E751
 P 6800 3500
-F 0 "#PWR031" H 6800 3250 50  0001 C CNN
+F 0 "#PWR041" H 6800 3250 50  0001 C CNN
 F 1 "GND" H 6800 3350 50  0000 C CNN
 F 2 "" H 6800 3500 60  0000 C CNN
@@
 Connection ~ 7700 2850
 $Comp
-L +3.3V #PWR032
+L +3.3V #PWR042
 U 1 1 5650E818
 P 7700 2200
-F 0 "#PWR032" H 7700 2050 50  0001 C CNN
+F 0 "#PWR042" H 7700 2050 50  0001 C CNN
 F 1 "+3.3V" H 7700 2340 50  0000 C CNN
 F 2 "" H 7700 2200 60  0000 C CNN
@@
 $EndComp
 $Comp
-L GND #PWR033
+L GND #PWR043
 U 1 1 5650E8BE
 P 7150 1700
-F 0 "#PWR033" H 7150 1450 50  0001 C CNN
+F 0 "#PWR043" H 7150 1450 50  0001 C CNN
 F 1 "GND" H 7150 1550 50  0000 C CNN
 F 2 "" H 7150 1700 60  0000 C CNN
@@
 Connection ~ 6400 1650
 $Comp
-L GND #PWR034
+L GND #PWR044
 U 1 1 5650F1ED
 P 6400 2150
-F 0 "#PWR034" H 6400 1900 50  0001 C CNN
+F 0 "#PWR044" H 6400 1900 50  0001 C CNN
 F 1 "GND" H 6400 2000 50  0000 C CNN
 F 2 "" H 6400 2150 60  0000 C CNN
@@
 Connection ~ 6450 3850
 $Comp
-L GND #PWR035
+L GND #PWR045
 U 1 1 5650F87C
 P 6450 4400
-F 0 "#PWR035" H 6450 4150 50  0001 C CNN
+F 0 "#PWR045" H 6450 4150 50  0001 C CNN
 F 1 "GND" H 6450 4250 50  0000 C CNN
 F 2 "" H 6450 4400 60  0000 C CNN
@@
 Connection ~ 2950 5400
 $Comp
-L GND #PWR036
+L GND #PWR046
 U 1 1 56634664
 P 2950 5850
-F 0 "#PWR036" H 2950 5600 50  0001 C CNN
+F 0 "#PWR046" H 2950 5600 50  0001 C CNN
 F 1 "GND" H 2950 5700 50  0000 C CNN
 F 2 "" H 2950 5850 50  0000 C CNN
@@
 	7200 3150 7200 2950
 $Comp
-L VCC #PWR037
+L VCC #PWR047
 U 1 1 56920678
 P 6400 1000
-F 0 "#PWR037" H 6400 850 50  0001 C CNN
+F 0 "#PWR047" H 6400 850 50  0001 C CNN
 F 1 "VCC" H 6400 1150 50  0000 C CNN
 F 2 "" H 6400 1000 50  0000 C CNN
@@
 $EndComp
 $Comp
-L VCC #PWR038
+L VCC #PWR048
 U 1 1 569206B9
 P 6800 1150
-F 0 "#PWR038" H 6800 1000 50  0001 C CNN
+F 0 "#PWR048" H 6800 1000 50  0001 C CNN
 F 1 "VCC" H 6800 1300 50  0000 C CNN
 F 2 "" H 6800 1150 50  0000 C CNN
@@
 $EndComp
 $Comp
-L VCC #PWR039
+L VCC #PWR049
 U 1 1 569207FD
 P 6450 3250
-F 0 "#PWR039" H 6450 3100 50  0001 C CNN
+F 0 "#PWR049" H 6450 3100 50  0001 C CNN
 F 1 "VCC" H 6450 3400 50  0000 C CNN
 F 2 "" H 6450 3250 50  0000 C CNN
@@
 $EndComp
 $Comp
-L VCC #PWR040
+L VCC #PWR050
 U 1 1 56920898
 P 2700 4800
-F 0 "#PWR040" H 2700 4650 50  0001 C CNN
+F 0 "#PWR050" H 2700 4650 50  0001 C CNN
 F 1 "VCC" H 2700 4950 50  0000 C CNN
 F 2 "" H 2700 4800 50  0000 C CNN
@@
 $EndComp
 $Comp
-L VCC #PWR041
+L VCC #PWR051
 U 1 1 569208D9
 P 3500 4650
-F 0 "#PWR041" H 3500 4500 50  0001 C CNN
+F 0 "#PWR051" H 3500 4500 50  0001 C CNN
 F 1 "VCC" H 3500 4800 50  0000 C CNN
 F 2 "" H 3500 4650 50  0000 C CNN
@@
 	1    0    0    -1
 $EndComp
+$Comp
+L TEST_1P W01
+U 1 1 5827C2E5
+P 5650 2650
+F 0 "W01" H 5650 2920 50  0000 C CNN
+F 1 "TEST_1P" H 5650 2850 50  0000 C CNN
+F 2 "MITEVT_TP:smd_test_pad" H 5850 2650 50  0001 C CNN
+F 3 "" H 5850 2650 50  0000 C CNN
+	1    5650 2650
+	1    0    0    -1
+$EndComp
+$Comp
+L TEST_1P W02
+U 1 1 5827C356
+P 5650 3050
+F 0 "W02" H 5650 3320 50  0000 C CNN
+F 1 "TEST_1P" H 5650 3250 50  0000 C CNN
+F 2 "MITEVT_TP:smd_test_pad" H 5850 3050 50  0001 C CNN
+F 3 "" H 5850 3050 50  0000 C CNN
+	1    5650 3050
+	-1   0    0    1
+$EndComp
+$Comp
+L TEST_1P W03
+U 1 1 5827C40C
+P 7850 2950
+F 0 "W03" H 7850 3220 50  0000 C CNN
+F 1 "TEST_1P" H 7850 3150 50  0000 C CNN
+F 2 "MITEVT_TP:smd_test_pad" H 8050 2950 50  0001 C CNN
+F 3 "" H 8050 2950 50  0000 C CNN
+	1    7850 2950
+	-1   0    0    1
+$EndComp
+Connection ~ 5650 2750
+Wire Wire Line
+	5650 3050 5650 2950
+Connection ~ 5650 2950
+Wire Wire Line
+	5650 2650 5650 2750
+Wire Wire Line
+	7850 2950 7850 2850
+Connection ~ 7850 2850
 $EndSCHEMATC
